File: electronics/BLDCM-Power/BLDCM-Power.kicad_pcb (KiCad board)
At the start: 4 copper layers, 32 x 32 mm, 60 parts, among them J1 501920-3001, J2 53048-0310, J3 505578-0460, J4 505578-0460, J5 FTSH-107-01-L-DV-K, J6 217179-0001, U1 INA240A1PWR, U10 BAT54S, U11 BAT54S, U12 BAT54S, U2 LDLN030G33R, U3 TMC6300-LA, U4 INA240A1PWR, U5 TCAN1462, U6 INA240A1PWR, U7 BAT54S, U8 LDO40LPU50RY, U9 TPS2115ADRB

Commit message: Refactor(schematic): Rename INA nets to CURR
Connections:
- net /INA.U renamed /CURR.U
- net /INA.V renamed /CURR.V
- net /INA.W renamed /CURR.W
